File: Hardware/ZED-F9P_NEO-D9S_Combo.sch (EAGLE design)
At the start: 97 parts, among them J1 ANTENNA-SMA-GROUNDEDEDGE_SMA, J2 Qwiic Right Angle, J3 USB Female Type C Connector, J4 Qwiic Right Angle, J6 USB Female Type C Connector, U1 U-BLOX_NEO-D9S-00B, U2 3.3V, U3 POWER-DIVIDER, U4 U-BLOX_ZED-F9P

Commit message: Add IC-16658 GNSS Power Divider. Delete New_parts.lbr
Parts:
- U3: device New_Parts:POWER-DIVIDER -> SparkFun-GPS:POWER-DIVIDER
Changed lines of the file:
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@@
 <part name="FRAME2" library="SparkFun-Aesthetics" deviceset="FRAME-LEDGER" device=""/>
 <part name="LOGO5" library="SparkFun-Aesthetics" deviceset="SPECIAL_INSTRUCTIONS" device="-ORDERING"/>
-<part name="U3" library="New_Parts" deviceset="POWER-DIVIDER" device=""/>
+<part name="U3" library="SparkFun-GPS" deviceset="POWER-DIVIDER" device=""/>
 <part name="U4" library="SparkFun-GPS" deviceset="U-BLOX_ZED-F9P" device=""/>
 <part name="R15" library="SparkFun-Resistors" deviceset="27OHM" device="-0603-1/10W-1%" value="27"/>

Commit message: Use RF Library copy of IC-16658
Parts:
- U3: device SparkFun-GPS:POWER-DIVIDER -> SparkFun-RF:POWER-DIVIDER
Changed lines of the file:
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@@
 <part name="FRAME2" library="SparkFun-Aesthetics" deviceset="FRAME-LEDGER" device=""/>
 <part name="LOGO5" library="SparkFun-Aesthetics" deviceset="SPECIAL_INSTRUCTIONS" device="-ORDERING"/>
-<part name="U3" library="SparkFun-GPS" deviceset="POWER-DIVIDER" device=""/>
+<part name="U3" library="SparkFun-RF" deviceset="POWER-DIVIDER" device=""/>
 <part name="U4" library="SparkFun-GPS" deviceset="U-BLOX_ZED-F9P" device=""/>
 <part name="R15" library="SparkFun-Resistors" deviceset="27OHM" device="-0603-1/10W-1%" value="27"/>

Commit message: x02 PCB - inverts RTK LED
Connections:
- net 3.3V: now also R27.2
- net GND: no longer LED2.C
- net RTK: now also LED2.C; no longer R27.2
Other:
- note added: "x02"
- note removed: "x01"
Changed lines of the file:
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@@
 <part name="LED2" library="SparkFun-LED" deviceset="LED-BLUE" device="0603" value="BLUE"/>
 <part name="RTK" library="SparkFun-Jumpers" deviceset="JUMPER-SMT_2_NC_TRACE" device="_SILK" package3d_urn="urn:adsk.eagle:package:39281/1" value="JUMPER-SMT_2_NC_TRACE_SILK"/>
-<part name="GND24" library="SparkFun-PowerSymbols" deviceset="GND" device=""/>
 <part name="R28" library="SparkFun-Resistors" deviceset="1KOHM" device="-0603-1/10W-1%" value="1k"/>
 <part name="LED3" library="SparkFun-LED" deviceset="LED-BLUE" device="0603" value="BLUE"/>
@@
 <part name="U$77" library="SparkX" deviceset="SPARKX-LOGO" device="4"/>
 <part name="U$78" library="SparkX" deviceset="SPARKX-LOGO" device="4"/>
+<part name="P+2" library="SparkFun-PowerSymbols" deviceset="3.3V" device=""/>
 </parts>
 <sheets>
 <sheet>
 <plain>
-<text x="420.624" y="7.366" size="2.54" layer="94" font="vector">x01</text>
+<text x="420.624" y="7.366" size="2.54" layer="94" font="vector">x02</text>
 <text x="187.96" y="210.82" size="1.778" layer="97" font="vector" align="center">7-bit unshifted I2C address: 0x43</text>
 <wire x1="0" y1="121.92" x2="68.58" y2="121.92" width="0.1524" layer="97" style="shortdash"/>
@@
 <attribute name="NAME" x="33.528" y="70.739" size="1.778" layer="95" font="vector" rot="R180"/>
 </instance>
-<instance part="GND24" gate="1" x="15.24" y="63.5" smashed="yes">
-<attribute name="VALUE" x="15.24" y="63.246" size="1.778" layer="96" font="vector" align="top-center"/>
-</instance>
 <instance part="R28" gate="G$1" x="48.26" y="50.8" smashed="yes">
 <attribute name="NAME" x="44.577" y="48.641" size="1.778" layer="95" font="vector" align="bottom-center"/>
@@
 <instance part="U$77" gate="G$1" x="383.54" y="48.26" smashed="yes"/>
 <instance part="U$78" gate="G$1" x="383.54" y="48.26" smashed="yes"/>
+<instance part="P+2" gate="G$1" x="55.88" y="71.12" smashed="yes">
+<attribute name="VALUE" x="55.88" y="73.914" size="1.778" layer="96" font="vector" align="bottom-center"/>
+</instance>
 </instances>
 <busses>
@@
 <wire x1="137.16" y1="246.38" x2="137.16" y2="248.92" width="0.1524" layer="91"/>
 </segment>
+<segment>
+<pinref part="R27" gate="G$1" pin="2"/>
+<wire x1="53.34" y1="68.58" x2="55.88" y2="68.58" width="0.1524" layer="91"/>
+<pinref part="P+2" gate="G$1" pin="3.3V"/>
+<wire x1="55.88" y1="68.58" x2="55.88" y2="71.12" width="0.1524" layer="91"/>
+</segment>
 </net>
 <net name="GND" class="0">
@@
 <wire x1="25.4" y1="243.84" x2="25.4" y2="241.3" width="0.1524" layer="91"/>
 <pinref part="C8" gate="G$1" pin="1"/>
-</segment>
-<segment>
-<pinref part="LED2" gate="G$1" pin="C"/>
-<wire x1="15.24" y1="68.58" x2="20.32" y2="68.58" width="0.1524" layer="91"/>
-<pinref part="GND24" gate="1" pin="GND"/>
-<wire x1="15.24" y1="66.04" x2="15.24" y2="68.58" width="0.1524" layer="91"/>
 </segment>
 <segment>
@@
 </segment>
 <segment>
-<label x="55.88" y="68.58" size="1.27" layer="95" xref="yes"/>
-<pinref part="R27" gate="G$1" pin="2"/>
-<wire x1="55.88" y1="68.58" x2="53.34" y2="68.58" width="0.1524" layer="91"/>
-</segment>
-<segment>
 <pinref part="J5" gate="J1" pin="4"/>
 <wire x1="175.26" y1="25.4" x2="172.72" y2="25.4" width="0.1524" layer="91"/>
 <label x="172.72" y="25.4" size="1.27" layer="95" rot="R180" xref="yes"/>
 </segment>
-</net>
+<segment>
+<pinref part="LED2" gate="G$1" pin="C"/>
+<wire x1="20.32" y1="68.58" x2="15.24" y2="68.58" width="0.1524" layer="91"/>
+<label x="15.24" y="68.58" size="1.27" layer="95" rot="R180" xref="yes"/>
+</segment>
+</net>
